File: ThermocoupleLogger.kicad_pcb (KiCad board)
At the start: 2 copper layers, 88.9 x 72.4 mm, 80 parts, among them J1 Barrel_Jack, P1 CONN_02X03, Q1 BS250, Q2 BD139, SW1 SW_Push, SW2 SW_Push, U1 LM3940, U10 TC_Connector, U11 ADG407, U12 I2C_20x4_DISPLAY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

Commit message: Commit2
Parts:
- removed the REF** at (100.1, 127.8)
Other:
- board text removed: "TEST"
Changed lines of the file:
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@@
   (general
     (thickness 1.6)
-    (drawings 22)
+    (drawings 21)
     (tracks 494)
     (zones 0)
-    (modules 80)
+    (modules 79)
     (nets 83)
   )
@@
     (add_net "Net-(BT2-Pad1)")
   )
-  (module Mounting_Holes:MountingHole_5.5mm (layer F.Cu)
-    (at 100.076 127.762)
-    (descr "Mounting Hole 5.5mm, no annular")
-    (tags "mounting hole 5.5mm no annular")
-    (fp_text reference REF** (at 0 -6.5) (layer F.SilkS)
-      (effects (font (size 1 1) (thickness 0.15)))
-    )
-    (fp_text value MountingHole_5.5mm (at 0 6.5) (layer F.Fab)
-      (effects (font (size 1 1) (thickness 0.15)))
-    )
-    (fp_circle (center 0 0) (end 5.5 0) (layer Cmts.User) (width 0.15))
-    (fp_circle (center 0 0) (end 5.75 0) (layer F.CrtYd) (width 0.05))
-    (pad 1 np_thru_hole circle (at 0 0) (size 5.5 5.5) (drill 5.5) (layers *.Cu *.Mask))
-  )
   (module Mounting_Holes:MountingHole_3.2mm_M3 (layer F.Cu)
     (at 97.79 76.2)
@@
     )
   )
-  (gr_text TEST (at 167.513 76.073) (layer F.Cu)
-    (effects (font (size 1.5 1.5) (thickness 0.3)))
-  )
   (gr_text "©2017, JP Enterprises" (at 171.704 125.984 90) (layer F.SilkS)

Commit message: Amend3
Parts:
- added REF**: MountingHole_5.5mm, Mounting_Holes:MountingHole_5.5mm, F.Cu at (168.9, 77.5)
Changed lines of the file:
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@@
     (tracks 494)
     (zones 0)
-    (modules 79)
+    (modules 80)
     (nets 83)
   )
@@
     (add_net "Net-(BT2-Pad1)")
   )
+  (module Mounting_Holes:MountingHole_5.5mm (layer F.Cu)
+    (at 168.91 77.47)
+    (descr "Mounting Hole 5.5mm, no annular")
+    (tags "mounting hole 5.5mm no annular")
+    (fp_text reference REF** (at 0 -6.5) (layer F.SilkS)
+      (effects (font (size 1 1) (thickness 0.15)))
+    )
+    (fp_text value MountingHole_5.5mm (at 0 6.5) (layer F.Fab)
+      (effects (font (size 1 1) (thickness 0.15)))
+    )
+    (fp_circle (center 0 0) (end 5.5 0) (layer Cmts.User) (width 0.15))
+    (fp_circle (center 0 0) (end 5.75 0) (layer F.CrtYd) (width 0.05))
+    (pad 1 np_thru_hole circle (at 0 0) (size 5.5 5.5) (drill 5.5) (layers *.Cu *.Mask))
+  )
   (module Mounting_Holes:MountingHole_3.2mm_M3 (layer F.Cu)

Commit message: Test edits
Parts:
- removed QR*****: ca9ed02408, jp_personal:ca9ed02408
- moved REF** 70.5 mm to (99.6, 90.4)
- moved REF*** 9.81 mm to (169.7, 92.5)
- moved U13 4.66 mm to (172.7, 123.4)
- turned REF** to 270 degrees

Commit message: Random edit
Parts:
- moved REF** 70.2 mm to (169.5, 96.8)
- moved REF** 6.41 mm to (179.8, 97.1)
- moved REF*** 5.80 mm to (171.5, 87.0)
